File: LinTech-UKNC/KiCad/LinTech-UKNC-board.sch (KiCad schematic (older format))
At the start: 34 parts, among them J1 K2, Q1 КТ315Г, Y1 12MHz

Commit message: BOM
Parts:
- DD1: value 74LS00 -> i8031
- DD13: value 580DD55A -> 580VV55A
- J1: value K2 -> ~
- LAN1: value Conn_02x05_Odd_Even -> ОНП-КГ-56-10/33х7,4-В53
- WS1: value Conn_02x07_Counter_Clockwise -> ~
Changed lines of the file:
@@
 P 2350 3400
 F 0 "J1" H 2400 4925 50  0000 C CNN
-F 1 "K2" H 2400 4926 50  0001 C CNN
+F 1 "~" H 2400 4926 50  0001 C CNN
 F 2 "Lib-UKNC:UKNC-CA" H 2350 3400 50  0001 C CNN
 F 3 "~" H 2350 3400 50  0001 C CNN
@@
 U 1 1 6671ACA6
 P 7500 3025
-F 0 "DD1" H 7500 4514 50  0000 C CNN
-F 1 "74LS00" H 7500 4515 50  0001 C CNN
+F 0 "DD1" H 7500 4600 50  0000 C CNN
+F 1 "i8031" H 7500 4515 50  0000 C CNN
 F 2 "Lib-UKNC:DIP-40_W15.24mm" H 7850 1775 50  0001 C CNN
 F 3 "http://www.ti.com/lit/gpn/sn74ls00" H 7500 3025 50  0001 C CNN
@@
 P 17525 3200
 F 0 "DD13" H 17525 4981 50  0000 C CNN
-F 1 "580DD55A" H 17525 4890 50  0000 C CNN
+F 1 "580VV55A" H 17525 4890 50  0000 C CNN
 F 2 "Lib-UKNC:DIP-40_W15.24mm" H 17525 3500 50  0001 C CNN
 F 3 "http://aturing.umcs.maine.edu/~meadow/courses/cos335/Intel8255A.pdf" H 17525 3500 50  0001 C CNN
@@
 P 12225 11625
 F 0 "WS1" H 12275 12050 50  0000 C CNN
-F 1 "Conn_02x07_Counter_Clockwise" H 12275 12051 50  0001 C CNN
+F 1 "~" H 12275 12051 50  0001 C CNN
 F 2 "Lib-UKNC:DIP-14_W7.62mm" H 12225 11625 50  0001 C CNN
 F 3 "~" H 12225 11625 50  0001 C CNN
@@
 P 15600 12425
 F 0 "LAN1" H 15650 12750 50  0000 C CNN
-F 1 "Conn_02x05_Odd_Even" H 15650 12751 50  0001 C CNN
+F 1 "ОНП-КГ-56-10/33х7,4-В53" H 15650 12751 50  0001 C CNN
 F 2 "Connector_PinHeader_2.54mm:PinHeader_2x05_P2.54mm_Horizontal" H 15600 12425 50  0001 C CNN
 F 3 "~" H 15600 12425 50  0001 C CNN
