File: LinTech-GM/KiCad/LinTech-GM-board_NC-ACM-2.2.sch (KiCad schematic (older format))
At the start: 78 parts, among them Q1 12000 KHz, X1 Conn_01x08_Male, X2 Conn_01x08_Male, X3 Conn_01x08_Male, X4 Conn_01x08_Male, X7 Conn_02x03_Counter_Clockwise

Commit message: Initial 2
Parts:
- R1: value R1 -> 3.3K
- R11: value R11 -> K10
- R12: value R12 -> 3.3K
- R13, R3: value R -> 470
- R14: value R14 -> 47K
- R2, R4: value R -> 1K
- R5: value R5 -> 150
- R6: value R6 -> 91R
- R7: value R7 -> 91R
- R9: value R9 -> 470 ??
- VD1: value VD1 -> КД522Б
- VD2: value VD2 -> КД522Б
- VD3: value VD3 -> КД522Б
- VD4: value ~ -> КД522Б
- VT1, VT4: value КТ315Б -> КТ646Б; symbol Connector:Conn_01x03_Male -> Device:Q_NPN_ECB
- VT5: value КТ315Б -> КТ313Б ?; symbol Connector:Conn_01x03_Male -> Device:Q_PNP_CBE
Connections:
- net +5V: now also VD1.1 (K), VD2.1 (K), VD3.1 (K), VD4.2 (A), VT3.2 (C); no longer VD1.2 (A), VD2.2 (A), VD3.2 (A), VD4.1 (K)
- net DD10_Out11: now also VD1.2 (A); no longer VD1.1 (K)
- net DD5-OE: now also DD3.7 (Q0a)
- net at C3.1, R11.1, R12.1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: now also VD3.2 (A); no longer VD3.1 (K)
- net at DD10.1, DD10.2, R3.2: now also VD2.2 (A); no longer VD2.1 (K)
- net at R14.2, VT5.3 (E): now also VD4.1 (K); no longer VD4.2 (A)
- net at R9.1: now also R10.1, VT4.3 (B)
Other:
- note added: "???\nкончается переходным\nпод DD3. \nВнешнее ПЗУ прошивки?"
- note removed: "???"
- note removed: "??? VT4 1,2,3"
- note removed: "??? Кудато сюда\nприходит +5"
- note removed: "кончается переходным\nпод DD3. \nВнешнее ПЗУ прошивки?"
- moved on the sheet: C12, C3, DD10A, DD10D, LD1, R1, R10, R11, R12, R13, R14, R3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

Commit message: BOM
Parts:
- C12: value C12 -> ~
- C3: value C3 -> ~
- DD5: value Conn_02x12_Counter_Clockwise -> Socket DIP24
- NR1: value R_Network09 -> 3.3K ?
- NR2: value R_Network09 -> ~
- R10: value R10 -> ~
- R9: value 470 ?? -> 470
- SAjp1, SAjp2, SAjp4, SAjp5, SAjp7, SAjp8: value Jumper_NO_Small -> ~
- SAjp3, SAjp6: value Jumper_NC_Small -> ~
- VT5: value КТ313Б ? -> КТ313Б
- X1, X2, X3, X4: value Conn_01x08_Male -> ~
- XA.1, XA.2: value Conn_01x31_Male -> ~
Changed lines of the file:
@@
 P 5475 10700
 F 0 "XA.2" H 5675 12350 50  0000 R CNN
-F 1 "Conn_01x31_Male" H 5447 10633 50  0001 R CNN
+F 1 "~" H 5447 10633 50  0001 R CNN
 F 2 "Connector_PinHeader_2.54mm:PinHeader_1x31_P2.54mm_Vertical" H 5475 10700 50  0001 C CNN
 F 3 "~" H 5475 10700 50  0001 C CNN
@@
 P 5825 10700
 F 0 "XA.1" H 5925 12350 50  0000 C CNN
-F 1 "Conn_01x31_Male" H 5933 12290 50  0001 C CNN
+F 1 "~" H 5933 12290 50  0001 C CNN
 F 2 "Connector_PinHeader_2.54mm:PinHeader_1x31_P2.54mm_Vertical" H 5825 10700 50  0001 C CNN
 F 3 "~" H 5825 10700 50  0001 C CNN
@@
 P 5450 5325
 F 0 "X1" H 5422 5253 50  0000 R CNN
-F 1 "Conn_01x08_Male" H 5558 5715 50  0001 C CNN
+F 1 "~" H 5558 5715 50  0001 C CNN
 F 2 "lib:PinHeader_1x08_P2.54mm_Vertical" H 5450 5325 50  0001 C CNN
 F 3 "~" H 5450 5325 50  0001 C CNN
@@
 P 5450 4375
 F 0 "X2" H 5422 4303 50  0000 R CNN
-F 1 "Conn_01x08_Male" H 5558 4765 50  0001 C CNN
+F 1 "~" H 5558 4765 50  0001 C CNN
 F 2 "lib:PinHeader_1x08_P2.54mm_Vertical" H 5450 4375 50  0001 C CNN
 F 3 "~" H 5450 4375 50  0001 C CNN
@@
 P 13775 2400
 F 0 "DD5" H 13825 3117 50  0000 C CNN
-F 1 "Conn_02x12_Counter_Clockwise" H 13825 3026 50  0001 C CNN
+F 1 "Socket DIP24" H 13825 3026 50  0001 C CNN
 F 2 "lib:DIP-24_W15.24mm_Socket" H 13775 2400 50  0001 C CNN
 F 3 "~" H 13775 2400 50  0001 C CNN
@@
 P 6275 7750
 F 0 "NR1" V 5750 7750 50  0000 C CNN
-F 1 "R_Network09" V 5749 7750 50  0001 C CNN
+F 1 "3.3K ?" V 5749 7750 50  0001 C CNN
 F 2 "Resistor_THT:R_Array_SIP10" V 6850 7750 50  0001 C CNN
 F 3 "http://www.vishay.com/docs/31509/csc.pdf" H 6275 7750 50  0001 C CNN
@@
 P 7925 4525
 F 0 "NR2" V 7400 4525 50  0000 C CNN
-F 1 "R_Network09" V 7399 4525 50  0001 C CNN
+F 1 "~" V 7399 4525 50  0001 C CNN
 F 2 "Resistor_THT:R_Array_SIP10" V 8500 4525 50  0001 C CNN
 F 3 "http://www.vishay.com/docs/31509/csc.pdf" H 7925 4525 50  0001 C CNN
@@
 P 7125 5475
 F 0 "X4" H 7275 5925 50  0000 R CNN
-F 1 "Conn_01x08_Male" H 7233 5865 50  0001 C CNN
+F 1 "~" H 7233 5865 50  0001 C CNN
 F 2 "lib:PinHeader_1x08_P2.54mm_Vertical" H 7125 5475 50  0001 C CNN
 F 3 "~" H 7125 5475 50  0001 C CNN
@@
 P 7125 4425
 F 0 "X3" H 7325 4850 50  0000 R CNN
-F 1 "Conn_01x08_Male" H 7233 4815 50  0001 C CNN
+F 1 "~" H 7233 4815 50  0001 C CNN
 F 2 "lib:PinHeader_1x08_P2.54mm_Vertical" H 7125 4425 50  0001 C CNN
 F 3 "~" H 7125 4425 50  0001 C CNN
@@
 P 20075 5300
 F 0 "R9" H 20000 5275 50  0000 R CNN
-F 1 "470 ?? " H 20005 5345 50  0000 R CNN
+F 1 "470" H 20005 5345 50  0000 R CNN
 F 2 "lib:R_Axial_DIN0207_L6.3mm_D2.5mm_P10.16mm_Horizontal" V 20005 5300 50  0001 C CNN
 F 3 "~" H 20075 5300 50  0001 C CNN
@@
 P 20075 5800
 F 0 "R10" H 20145 5800 50  0000 L CNN
-F 1 "R10" H 20005 5845 50  0001 R CNN
+F 1 "~" H 20005 5845 50  0001 R CNN
 F 2 "lib:R_Axial_DIN0207_L6.3mm_D2.5mm_P10.16mm_Horizontal" V 20005 5800 50  0001 C CNN
 F 3 "~" H 20075 5800 50  0001 C CNN
@@
 P 18050 5625
 F 0 "C3" H 17950 5725 50  0000 C CNN
-F 1 "C3" V 17889 5625 50  0001 C CNN
+F 1 "~" V 17889 5625 50  0001 C CNN
 F 2 "lib:C_Disc_D5.0mm_W2.5mm_P5.00mm" H 18088 5475 50  0001 C CNN
 F 3 "~" H 18050 5625 50  0001 C CNN
@@
 P 18475 6275
 F 0 "VT5" H 18900 6325 70  0000 R CNN
-F 1 "КТ313Б ?" H 18725 6225 70  0000 L CNN
+F 1 "КТ313Б" H 18725 6225 70  0000 L CNN
 F 2 "Package_TO_SOT_THT:TO-92" H 18475 6275 70  0001 C CNN
 F 3 "" H 18475 6275 70  0001 C CNN
@@
 P 21075 2025
 F 0 "C12" V 20900 2025 50  0000 C CNN
-F 1 "C12" V 20914 2025 50  0001 C CNN
+F 1 "~" V 20914 2025 50  0001 C CNN
 F 2 "lib:C_Disc_D5.0mm_W2.5mm_P5.00mm" H 21113 1875 50  0001 C CNN
 F 3 "~" H 21075 2025 50  0001 C CNN
@@
 P 5225 7350
 F 0 "SAjp1" H 5225 7535 50  0001 C CNN
-F 1 "Jumper_NO_Small" H 5225 7444 50  0001 C CNN
+F 1 "~" H 5225 7444 50  0001 C CNN
 F 2 "lib:Jumper_P2.54mm_Open" H 5225 7350 50  0001 C CNN
 F 3 "~" H 5225 7350 50  0001 C CNN
@@
 P 5225 7450
 F 0 "SAjp2" H 5225 7635 50  0001 C CNN
-F 1 "Jumper_NO_Small" H 5225 7544 50  0001 C CNN
+F 1 "~" H 5225 7544 50  0001 C CNN
 F 2 "lib:Jumper_P2.54mm_Open" H 5225 7450 50  0001 C CNN
 F 3 "~" H 5225 7450 50  0001 C CNN
@@
 P 5225 7650
 F 0 "SAjp4" H 5225 7835 50  0001 C CNN
-F 1 "Jumper_NO_Small" H 5225 7744 50  0001 C CNN
+F 1 "~" H 5225 7744 50  0001 C CNN
 F 2 "lib:Jumper_P2.54mm_Open" H 5225 7650 50  0001 C CNN
 F 3 "~" H 5225 7650 50  0001 C CNN
@@
 P 5225 7750
 F 0 "SAjp5" H 5225 7935 50  0001 C CNN
-F 1 "Jumper_NO_Small" H 5225 7844 50  0001 C CNN
+F 1 "~" H 5225 7844 50  0001 C CNN
 F 2 "lib:Jumper_P2.54mm_Open" H 5225 7750 50  0001 C CNN
 F 3 "~" H 5225 7750 50  0001 C CNN
@@
 P 5225 7950
 F 0 "SAjp7" H 5225 8135 50  0001 C CNN
-F 1 "Jumper_NO_Small" H 5225 8044 50  0001 C CNN
+F 1 "~" H 5225 8044 50  0001 C CNN
 F 2 "lib:Jumper_P2.54mm_Open" H 5225 7950 50  0001 C CNN
 F 3 "~" H 5225 7950 50  0001 C CNN
@@
 P 5225 8050
 F 0 "SAjp8" H 5225 8235 50  0001 C CNN
-F 1 "Jumper_NO_Small" H 5225 8144 50  0001 C CNN
+F 1 "~" H 5225 8144 50  0001 C CNN
 F 2 "lib:Jumper_P2.54mm_Open" H 5225 8050 50  0001 C CNN
 F 3 "~" H 5225 8050 50  0001 C CNN
@@
 P 5225 7550
 F 0 "SAjp3" H 5225 7762 50  0001 C CNN
-F 1 "Jumper_NC_Small" H 5225 7671 50  0001 C CNN
+F 1 "~" H 5225 7671 50  0001 C CNN
 F 2 "lib:Jumper_P2.54mm_Close" H 5225 7550 50  0001 C CNN
 F 3 "~" H 5225 7550 50  0001 C CNN
@@
 P 5225 7850
 F 0 "SAjp6" H 5225 8062 50  0001 C CNN
-F 1 "Jumper_NC_Small" H 5225 7971 50  0001 C CNN
+F 1 "~" H 5225 7971 50  0001 C CNN
 F 2 "lib:Jumper_P2.54mm_Close" H 5225 7850 50  0001 C CNN
 F 3 "~" H 5225 7850 50  0001 C CNN

Commit message: Update GM schematic, README, split LInTech software archive
Parts:
- C1, C2: value C -> 18pF
- C12: value ~ -> 0.15 мкФ
- C3: value ~ -> 1нФ ?
- CF1, CF10, CF2, CF3, CF4, CF5, CF6, CF7, CF8, CF9: value C -> 150nF
- LD1: value LD1 -> LED Red 4mm
- LD2: value LD2 -> LED Red 4mm
- R10: value ~ -> 150
Changed lines of the file:
@@
 P 1950 13600
 F 0 "CF2" V 1698 13600 50  0000 C CNN
-F 1 "C" V 1789 13600 50  0000 C CNN
+F 1 "150nF" V 1789 13600 50  0000 C CNN
 F 2 "lib:C_Disc_D5.0mm_W2.5mm_P5.00mm" H 1988 13450 50  0001 C CNN
 F 3 "~" H 1950 13600 50  0001 C CNN
@@
 P 1950 14025
 F 0 "CF3" V 1698 14025 50  0000 C CNN
-F 1 "C" V 1789 14025 50  0000 C CNN
+F 1 "150nF" V 1789 14025 50  0000 C CNN
 F 2 "lib:C_Disc_D5.0mm_W2.5mm_P5.00mm" H 1988 13875 50  0001 C CNN
 F 3 "~" H 1950 14025 50  0001 C CNN
@@
 P 3125 13250
 F 0 "CF6" V 2873 13250 50  0000 C CNN
-F 1 "C" V 2964 13250 50  0000 C CNN
+F 1 "150nF" V 2964 13250 50  0000 C CNN
 F 2 "lib:C_Disc_D5.0mm_W2.5mm_P5.00mm" H 3163 13100 50  0001 C CNN
 F 3 "~" H 3125 13250 50  0001 C CNN
@@
 P 3125 13650
 F 0 "CF7" V 2873 13650 50  0000 C CNN
-F 1 "C" V 2964 13650 50  0000 C CNN
+F 1 "150nF" V 2964 13650 50  0000 C CNN
 F 2 "lib:C_Disc_D5.0mm_W2.5mm_P5.00mm" H 3163 13500 50  0001 C CNN
 F 3 "~" H 3125 13650 50  0001 C CNN
@@
 P 3125 14050
 F 0 "CF8" V 3377 14050 50  0000 C CNN
-F 1 "C" V 3286 14050 50  0000 C CNN
+F 1 "150nF" V 3286 14050 50  0000 C CNN
 F 2 "lib:C_Disc_D5.0mm_W2.5mm_P5.00mm" H 3163 13900 50  0001 C CNN
 F 3 "~" H 3125 14050 50  0001 C CNN
@@
 P 3125 14450
 F 0 "CF9" V 2873 14450 50  0000 C CNN
-F 1 "C" V 2964 14450 50  0000 C CNN
+F 1 "150nF" V 2964 14450 50  0000 C CNN
 F 2 "lib:C_Disc_D5.0mm_W2.5mm_P5.00mm" H 3163 14300 50  0001 C CNN
 F 3 "~" H 3125 14450 50  0001 C CNN
@@
 P 3125 14850
 F 0 "CF10" V 2873 14850 50  0000 C CNN
-F 1 "C" V 2964 14850 50  0000 C CNN
+F 1 "150nF" V 2964 14850 50  0000 C CNN
 F 2 "lib:C_Disc_D5.0mm_W2.5mm_P5.00mm" H 3163 14700 50  0001 C CNN
 F 3 "~" H 3125 14850 50  0001 C CNN
@@
 P 3100 3500
 F 0 "C1" V 2848 3500 50  0000 C CNN
-F 1 "C" V 2939 3500 50  0000 C CNN
+F 1 "18pF" V 2939 3500 50  0000 C CNN
 F 2 "lib:C_Disc_D5.0mm_W2.5mm_P5.00mm" H 3138 3350 50  0001 C CNN
 F 3 "~" H 3100 3500 50  0001 C CNN
@@
 U 1 1 652B608C
 P 3100 3800
-F 0 "C2" V 2848 3800 50  0000 C CNN
-F 1 "C" V 2939 3800 50  0000 C CNN
+F 0 "C2" V 2925 3800 50  0000 C CNN
+F 1 "18pF" V 2850 3800 50  0000 C CNN
 F 2 "lib:C_Disc_D5.0mm_W2.5mm_P5.00mm" H 3138 3650 50  0001 C CNN
 F 3 "~" H 3100 3800 50  0001 C CNN
@@
 P 1950 13225
 F 0 "CF1" V 1698 13225 50  0000 C CNN
-F 1 "C" V 1789 13225 50  0000 C CNN
+F 1 "150nF" V 1789 13225 50  0000 C CNN
 F 2 "lib:C_Disc_D5.0mm_W2.5mm_P5.00mm" H 1988 13075 50  0001 C CNN
 F 3 "~" H 1950 13225 50  0001 C CNN
@@
 P 1950 14425
 F 0 "CF4" V 1698 14425 50  0000 C CNN
-F 1 "C" V 1789 14425 50  0000 C CNN
+F 1 "150nF" V 1789 14425 50  0000 C CNN
 F 2 "lib:C_Disc_D5.0mm_W2.5mm_P5.00mm" H 1988 14275 50  0001 C CNN
 F 3 "~" H 1950 14425 50  0001 C CNN
@@
 P 1950 14825
 F 0 "CF5" V 1698 14825 50  0000 C CNN
-F 1 "C" V 1789 14825 50  0000 C CNN
+F 1 "150nF" V 1789 14825 50  0000 C CNN
 F 2 "lib:C_Disc_D5.0mm_W2.5mm_P5.00mm" H 1988 14675 50  0001 C CNN
 F 3 "~" H 1950 14825 50  0001 C CNN
@@
 P 18425 4200
 F 0 "LD1" H 18418 4037 50  0000 C CNN
-F 1 "LD1" H 18418 4036 50  0001 C CNN
+F 1 "LED Red 4mm" H 18418 4036 50  0001 C CNN
 F 2 "LED_THT:LED_D4.0mm" H 18425 4200 50  0001 C CNN
 F 3 "~" H 18425 4200 50  0001 C CNN
@@
 P 3775 2150
 F 0 "LD2" H 3768 1987 50  0000 C CNN
-F 1 "LD2" H 3768 1986 50  0001 C CNN
+F 1 "LED Red 4mm" H 3768 1986 50  0001 C CNN
 F 2 "LED_THT:LED_D4.0mm" H 3775 2150 50  0001 C CNN
 F 3 "~" H 3775 2150 50  0001 C CNN
@@
 U 1 1 666206BB
 P 20075 5800
-F 0 "R10" H 20145 5800 50  0000 L CNN
-F 1 "~" H 20005 5845 50  0001 R CNN
+F 0 "R10" H 20150 5850 50  0000 L CNN
+F 1 "150" H 20300 5775 50  0000 R CNN
 F 2 "lib:R_Axial_DIN0207_L6.3mm_D2.5mm_P10.16mm_Horizontal" V 20005 5800 50  0001 C CNN
 F 3 "~" H 20075 5800 50  0001 C CNN
@@
 U 1 1 6667A531
 P 18050 5625
-F 0 "C3" H 17950 5725 50  0000 C CNN
-F 1 "~" V 17889 5625 50  0001 C CNN
+F 0 "C3" H 17825 5650 50  0000 C CNN
+F 1 "1нФ ?" H 17800 5575 50  0000 C CNN
 F 2 "lib:C_Disc_D5.0mm_W2.5mm_P5.00mm" H 18088 5475 50  0001 C CNN
 F 3 "~" H 18050 5625 50  0001 C CNN
@@
 U 1 1 6667AD04
 P 21075 2025
-F 0 "C12" V 20900 2025 50  0000 C CNN
-F 1 "~" V 20914 2025 50  0001 C CNN
+F 0 "C12" H 20875 2075 50  0000 C CNN
+F 1 "0.15 мкФ" H 20800 2000 50  0000 C CNN
 F 2 "lib:C_Disc_D5.0mm_W2.5mm_P5.00mm" H 21113 1875 50  0001 C CNN
 F 3 "~" H 21075 2025 50  0001 C CNN

Commit message: Fix footprint drill diameters
Parts:
- LD1, LD2: footprint LED_THT:LED_D4.0mm -> lib:LED_D4.0mm
- VT2, VT3: footprint Package_TO_SOT_THT:TO-92S_Wide -> lib:TO-92S_Wide
Changed lines of the file:
@@
 Rev "2.2"
 Comp "LInTech"
-Comment1 "gryphon@night-gryphon.ru"
-Comment2 "Reconstruction by Night_Gryphon"
-Comment3 ""
+Comment1 "https://github.com/nightgryphon/LInTech-network"
+Comment2 "gryphon@night-gryphon.ru"
+Comment3 "Reconstruction by Night_Gryphon"
 Comment4 "LInTech GM"
 $EndDescr
@@
 F 0 "LD1" H 18418 4037 50  0000 C CNN
 F 1 "LED Red 4mm" H 18418 4036 50  0001 C CNN
-F 2 "LED_THT:LED_D4.0mm" H 18425 4200 50  0001 C CNN
+F 2 "lib:LED_D4.0mm" H 18425 4200 50  0001 C CNN
 F 3 "~" H 18425 4200 50  0001 C CNN
 	1    18425 4200
@@
 F 0 "LD2" H 3768 1987 50  0000 C CNN
 F 1 "LED Red 4mm" H 3768 1986 50  0001 C CNN
-F 2 "LED_THT:LED_D4.0mm" H 3775 2150 50  0001 C CNN
+F 2 "lib:LED_D4.0mm" H 3775 2150 50  0001 C CNN
 F 3 "~" H 3775 2150 50  0001 C CNN
 	1    3775 2150
@@
 F 0 "VT2" H 20350 2125 70  0000 R CNN
 F 1 "КТ315Б" H 20150 2025 70  0000 L CNN
-F 2 "Package_TO_SOT_THT:TO-92S_Wide" H 19975 2075 70  0001 C CNN
+F 2 "lib:TO-92S_Wide" H 19975 2075 70  0001 C CNN
 F 3 "" H 19975 2075 70  0001 C CNN
 	1    19975 2075
@@
 F 0 "VT3" H 20375 5000 70  0000 R CNN
 F 1 "КТ315Б" H 20175 4900 70  0000 L CNN
-F 2 "Package_TO_SOT_THT:TO-92S_Wide" H 19975 4950 70  0001 C CNN
+F 2 "lib:TO-92S_Wide" H 19975 4950 70  0001 C CNN
 F 3 "" H 19975 4950 70  0001 C CNN
 	1    19975 4950

Commit message: Adjust test pads, track width, DB9
Parts:
- XA.1, XA.2: footprint Connector_PinHeader_2.54mm:PinHeader_1x31_P2.54mm_Vertical -> lib:PinHeader_1x31_P2.54mm_Vertical
Changed lines of the file:
@@
 F 0 "XA.2" H 5675 12350 50  0000 R CNN
 F 1 "~" H 5447 10633 50  0001 R CNN
-F 2 "Connector_PinHeader_2.54mm:PinHeader_1x31_P2.54mm_Vertical" H 5475 10700 50  0001 C CNN
+F 2 "lib:PinHeader_1x31_P2.54mm_Vertical" H 5475 10700 50  0001 C CNN
 F 3 "~" H 5475 10700 50  0001 C CNN
 	1    5475 10700
@@
 F 0 "XA.1" H 5925 12350 50  0000 C CNN
 F 1 "~" H 5933 12290 50  0001 C CNN
-F 2 "Connector_PinHeader_2.54mm:PinHeader_1x31_P2.54mm_Vertical" H 5825 10700 50  0001 C CNN
+F 2 "lib:PinHeader_1x31_P2.54mm_Vertical" H 5825 10700 50  0001 C CNN
 F 3 "~" H 5825 10700 50  0001 C CNN
 	1    5825 10700
